File: Hardware/OM_Landroid_MB/imu.kicad_sch (KiCad schematic)
At the start: 8 parts

Commit message: Weekend progress
Parts:
- removed JP10, JP11: I2C_OR_TTL, Jumper:SolderJumper-3_P1.3mm_Bridged12_Pad1.0x1.5mm, symbol Jumper:SolderJumper_3_Bridged12
- removed R14, R17: 4k7, Resistor_SMD:R_0805_2012Metric_Pad1.20x1.40mm_HandSolder, symbol Device:R
- removed WT901: Conn_02x06_Female, MyModules:WT901, symbol Connector_Generic:Conn_02x06_Row_Letter_First
Connections:
- no-connect marks 8 -> 4
Other:
- moved on the sheet: AC1201, C24, C26
