File: Hardware/OM_Landroid_MB/OM Landroid MB.kicad_pcb (KiCad board)
At the start: 2 copper layers, 83.8 x 88.9 mm, 126 parts, among them IC1 74ALVC164245DGG,11, IC2 TSC101CILT, IC3 MAX20405AFOF_VY+T, J1 Conn_01x02_Pin, J11 Conn_01x03_Male, J12 Conn_01x03_Male, J13 Conn_01x03_Male, J14 Conn_01x03_Male, J17 Conn_01x02, J19 Conn_01x04, J2 Conn_02x04_Top_Bottom, J21 Raspberry_Pi_2_3, J22 Conn_02x04_Odd_Even, J3 Conn_01x02, J5 Conn_01x04, J51 Conn_01x05_Socket, J52 Conn_01x05_Socket, J6 Conn_01x04, M1 Fan, Q3 BSS138, Q5 BSS138, Q6 Q_PMOS_GDS, SW1 MK-11C04-G013, U10 74HC4051, U11 Pico, U2 MCP604, U3 SIP32509DT, U4 xESC2, U5 xESC2, U6 xESC2, U7 SN74LV1T34DBV, U9 74HC4051

Commit message: Add files via upload
Parts:
- J51: footprint Connector_JST:JST_XH_B5B-XH-A_1x05_P2.50mm_Vertical -> Connector_JST:JST_XH_B4B-XH-A_1x04_P2.50mm_Vertical
- JC1, JL1, JR1: footprint Connector_Molex:Molex_KK-254_AE-6410-03A_1x03_P2.54mm_Vertical -> Landroid_Motor_Conn:TE_179839
- moved JR1 11.8 mm to (241.7, 96.4)
- moved JL1 8.32 mm to (241.9, 41.3)
- moved JC1 8.10 mm to (241.8, 71.6)
- moved J51 1.25 mm to (118.9, 86.9)
Connections:
- J51 pad 2: +3.3V -> /RaspberryPi/UART1_TXD
- J51 pad 4: /RaspberryPi/UART1_TXD -> GND

Commit message: Weekend progress
Parts:
- removed C10: DNP, Capacitor_SMD:CP_Elec_10x12.5
- removed D17: DNP, Diode_SMD:D_0402_1005Metric_Pad0.77x0.64mm_HandSolder
- removed JP10, JP11: I2C_OR_TTL, Jumper:SolderJumper-3_P1.3mm_Bridged12_Pad1.0x1.5mm
- removed JP4, JP5: SolderJumper_3_Bridged12, Jumper:SolderJumper-3_P1.3mm_Bridged12_Pad1.0x1.5mm
- removed R11: 53k6 1%, Resistor_SMD:R_0805_2012Metric_Pad1.20x1.40mm_HandSolder
- removed R12: 10k, Resistor_SMD:R_0805_2012Metric_Pad1.20x1.40mm_HandSolder
- removed R14, R17: 4k7, Resistor_SMD:R_0805_2012Metric_Pad1.20x1.40mm_HandSolder
- removed WT901: Conn_02x06_Female, MyModules:WT901
- J21: footprint RPi_c:RPi_40Pin_Fan_Courtyard -> Connector_PinSocket_2.54mm:PinSocket_2x20_P2.54mm_Vertical
- J51: footprint Connector_JST:JST_XH_B4B-XH-A_1x04_P2.50mm_Vertical -> Connector_JST:JST_XH_B4B-XH-AM_1x04_P2.50mm_Vertical
- JC1, JL1, JR1: footprint Landroid_Motor_Conn:TE_179839 -> Connector_Molex:Molex_KK-254_AE-6410-03A_1x03_P2.54mm_Vertical
- R8: value DNP -> 5k
- moved Q6 108.1 mm to (71.5, 139.2)
- moved IC2 107.4 mm to (62.4, 127.5)
- moved R28 107.4 mm to (70.7, 121.2)
- moved TP5 107.4 mm to (66.6, 126.9)
- moved C5 107.4 mm to (65.3, 113.6)
- moved Q5 107.4 mm to (76.7, 122.4)
- moved D13 107.4 mm to (60.2, 112.9)
- moved R26 107.4 mm to (70.7, 118.4)
- moved R27 107.4 mm to (70.7, 123.7)
- moved R51 107.4 mm to (64.0, 120.5)
- moved J17 89.1 mm to (66.5, 49.6), turned to -90 degrees
- moved SW1 79.9 mm to (130.4, 158.2), turned to 0 degrees
- moved JP8 59.2 mm to (146.6, 146.8)
- moved D1 56.5 mm to (121.4, 150.0)
- moved M1 56.5 mm to (122.7, 156.3)
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Connections:
- net /IMU/TX renamed /IMU/~{CS}
- C16 pad 1: +5V -> GND
- C16 pad 2: GND -> +5V
- C18 pad 1: +5V -> GND
- C18 pad 2: GND -> +5V
- C19 pad 1: +5V -> GND
- C19 pad 2: GND -> +5V
- C20 pad 1: +5V -> GND
- C20 pad 2: GND -> +5V
- C21 pad 1: +5V -> GND
- C21 pad 2: GND -> +5V
- C22 pad 1: +5V -> GND
- C22 pad 2: GND -> +5V
- IC1 pad 16: unconnected-(IC1-2B2-Pad16) -> /RobotConnectors/USS_1_TRIGGER_5V
- IC1 pad 19: /RobotConnectors/USS_1_TRIGGER_5V -> unconnected-(IC1-2B4-Pad19)
- IC1 pad 2: /RobotConnectors/USS_1_ECHO_5V -> /RobotConnectors/USS_2_ECHO_5V
- IC1 pad 3: /RobotConnectors/USS_2_ECHO_5V -> /RobotConnectors/USS_1_ECHO_5V
- IC1 pad 30: /RobotConnectors/USS_1_TRIGGER -> GND
- IC1 pad 33: GND -> /RobotConnectors/USS_1_TRIGGER
- IC1 pad 40: /RobotConnectors/HALL_SWITCH_4 -> /RobotConnectors/HALL_SWITCH_2
- IC1 pad 41: /RobotConnectors/HALL_SWITCH_3 -> /RobotConnectors/HALL_SWITCH_1
- IC1 pad 43: /RobotConnectors/HALL_SWITCH_2 -> /RobotConnectors/HALL_SWITCH_3
- IC1 pad 44: /RobotConnectors/HALL_SWITCH_1 -> /RobotConnectors/HALL_SWITCH_4
- IC1 pad 46: /RobotConnectors/USS_2_ECHO -> /RobotConnectors/USS_1_ECHO
- IC1 pad 47: /RobotConnectors/USS_1_ECHO -> /RobotConnectors/USS_2_ECHO
- IC1 pad 5: /RobotConnectors/HALL_SWITCH_1_5V -> /RobotConnectors/HALL_SWITCH_4_5V
- IC1 pad 6: /RobotConnectors/HALL_SWITCH_2_5V -> /RobotConnectors/HALL_SWITCH_3_5V
- IC1 pad 8: /RobotConnectors/HALL_SWITCH_3_5V -> /RobotConnectors/HALL_SWITCH_1_5V
- IC1 pad 9: /RobotConnectors/HALL_SWITCH_4_5V -> /RobotConnectors/HALL_SWITCH_2_5V
- IC3 pad 10: GND -> Net-(IC3-GND)
- IC3 pad 12: Net-(IC3-FB_1) -> Net-(IC3-BIAS)
- IC3 pad 16: Net-(IC3-SYNC) -> Net-(IC3-GND)
- IC3 pad 17: Net-(IC3-SYNCOUT_1) -> unconnected-(IC3-SYNCOUT_1-Pad17)
- J11 pad 2: /RobotConnectors/HALL_SWITCH_1_5V -> /RobotConnectors/HALL_SWITCH_4_5V
- J12 pad 2: /RobotConnectors/HALL_SWITCH_2_5V -> /RobotConnectors/HALL_SWITCH_3_5V
- J13 pad 2: /RobotConnectors/HALL_SWITCH_3_5V -> /RobotConnectors/HALL_SWITCH_1_5V
- J14 pad 2: /RobotConnectors/HALL_SWITCH_4_5V -> /RobotConnectors/HALL_SWITCH_2_5V
- R13 pad 1: Net-(J52-Pin_4) -> Net-(J52-Pin_3)
- R7 pad 1: Net-(J52-Pin_3) -> Net-(J52-Pin_4)
Routing:
- net GND: track 0.00 -> 1218.7 mm, vias 0 -> 27
- net +5V: track 0.00 -> 891.8 mm, vias 0 -> 8
- net V_BATT: track 0.00 -> 480.1 mm
- net /ESCs/ML_RX: track 0.00 -> 205.8 mm, vias 0 -> 2
- net /ESCs/ML_TX: track 0.00 -> 204.4 mm
- net /ESCs/MC_RX: track 0.00 -> 162.6 mm
- net /ESCs/MC_TX: track 0.00 -> 160.6 mm
- net /ESCs/MR_TX: track 0.00 -> 132.8 mm, vias 0 -> 2
- net /ESCs/MR_RX: track 0.00 -> 115.5 mm, vias 0 -> 1
- net +3V3: track 0.00 -> 112.5 mm, vias 0 -> 2
- net /RobotConnectors/HALL_SWITCH_4: track 0.00 -> 98.5 mm
- net Net-(U11-GPIO10): track 0.00 -> 97.1 mm, vias 0 -> 2
- net /RobotConnectors/HALL_SWITCH_3: track 0.00 -> 96.9 mm
- net /RobotConnectors/HALL_SWITCH_2: track 0.00 -> 88.0 mm
- net /ESCs/ESC_SHUTDOWN: track 0.00 -> 87.8 mm, vias 0 -> 2
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Other:
- board size 83.8 x 88.9 mm -> 54.5 x 139.7 mm

Commit message: Daily update
Parts:
- moved R27 164.2 mm to (234.5, 135.3)
- moved Q6 161.2 mm to (232.4, 147.7)
- moved R28 159.6 mm to (229.2, 139.7)
- moved R26 159.4 mm to (229.2, 135.3), turned to 180 degrees
- moved Q5 158.7 mm to (234.6, 138.9), turned to -90 degrees
- moved R51 149.4 mm to (213.1, 130.8)
- moved D13 146.5 mm to (204.7, 137.4), turned to 180 degrees
- moved TP5 144.0 mm to (210.2, 136.9)
- moved IC2 142.1 mm to (204.5, 130.9), turned to 90 degrees
- moved C1 107.0 mm to (198.8, 137.3)
- moved D14 44.0 mm to (204.8, 134.7)
- moved C25 18.6 mm to (182.6, 139.6)
- moved D25 18.6 mm to (188.6, 136.3)
- moved U7 18.6 mm to (181.6, 134.9)
- moved JP8 10.1 mm to (156.5, 148.3)
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Routing:
- net /CHARGE_CURRENT: track 0.00 -> 71.4 mm
- net /RaspberryPi/POWER_EN: track 1.60 -> 69.4 mm, vias 0 -> 2
- net GND: track 1218.7 -> 1275.7 mm, vias 27 -> 29
- net +5V: track 891.8 -> 869.4 mm
- net /RobotConnectors/MosfetSwitch/VOUT: track 0.00 -> 20.5 mm
- net /RobotConnectors/ENABLE_CHARGE: track 0.00 -> 15.2 mm
- net Net-(J21-GPIO23): track 36.8 -> 44.3 mm
- net Net-(J21-GPIO25): track 49.1 -> 56.6 mm
- net Net-(Q5-D): track 0.00 -> 7.22 mm
- net Net-(J21-GPIO24): track 42.3 -> 49.5 mm
- net /RobotConnectors/CHARGE_SHUNT_MINUS: track 0.00 -> 4.30 mm
- net /RaspberryPi/UART0_RXD: track 45.7 -> 43.0 mm
- net Net-(Q5-G): track 0.00 -> 2.61 mm
- net /pico/V_IN: track 0.00 -> 1.60 mm
- net /pico/V_CHARGE: track 0.00 -> 1.60 mm
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
Commit message: Update 21.11.23
Parts:
- U11: footprint PicoW:Raspberry_Pi_Pico_SMT_THT -> PicoW:Raspberry_Pi_Pico_THT
- moved J17 103.5 mm to (169.0, 64.6)
- moved R43 100.5 mm to (192.7, 128.8), turned to 0 degrees
- moved C5 93.4 mm to (155.2, 88.6), turned to -90 degrees
- moved JP7 69.4 mm to (153.9, 154.2)
- moved TP5 54.0 mm to (156.2, 135.4)
- moved J19 53.9 mm to (165.2, 106.5), turned to -90 degrees
- moved D13 51.6 mm to (153.5, 131.2), turned to 0 degrees
- moved D14 46.4 mm to (158.6, 131.2)
- moved R42 44.6 mm to (197.4, 128.8), turned to 0 degrees
- moved R1 39.6 mm to (115.4, 98.5)
- moved R40 36.4 mm to (197.3, 125.8)
- moved R2 35.6 mm to (110.5, 98.5)
- moved R41 34.5 mm to (192.8, 125.9), turned to 0 degrees
- moved R18 32.6 mm to (184.6, 146.7), turned to 90 degrees
- moved D23 29.8 mm to (181.0, 143.8), turned to 180 degrees
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Routing:
- net GND: track 1275.7 -> 1646.2 mm, vias 29 -> 38
- net /RobotConnectors/ENABLE_CHARGE: track 15.2 -> 172.3 mm, vias 0 -> 6
- net /pico/V_CHARGE: track 1.60 -> 120.1 mm, vias 0 -> 2
- net /pico/V_IN: track 1.60 -> 118.2 mm, vias 0 -> 2
- net /RaspberryPi/PICO_SWDIO: track 1.60 -> 97.6 mm, vias 0 -> 4
- net /RobotConnectors/V_CHARGE: track 5.00 -> 94.7 mm, vias 0 -> 4
- net /RaspberryPi/PICO_RESET: track 1.60 -> 89.2 mm, vias 0 -> 2
- net /RaspberryPi/PICO_SWCLK: track 1.60 -> 85.0 mm, vias 0 -> 4
- net +3V3: track 112.5 -> 191.5 mm, vias 2 -> 8
- net +5V: track 869.4 -> 937.7 mm, vias 8 -> 12
- net V_BATT: track 480.1 -> 424.5 mm
- net /CHARGE_CURRENT: track 71.4 -> 125.4 mm, vias 0 -> 4
- net /RobotConnectors/CHARGE_SHUNT_PLUS: track 0.00 -> 53.5 mm, vias 0 -> 2
- net /RobotConnectors/V_BATTERY: track 25.6 -> 78.7 mm, vias 0 -> 4
- net /RaspberryPi/RASPI_FAN_ON: track 18.5 -> 68.7 mm, vias 0 -> 1
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- added copper zone on F.Cu, net +5V
- added copper zone on B.Cu, net GND
- added copper zone on F.Cu, net GND
- added copper zone on F.Cu, net Net-(IC3-BIAS)
- added copper zone on F.Cu, net Net-(IC3-LX_1)
- added copper zone on F.Cu, net Net-(IC3-PGOOD)
- added copper zone on F.Cu, net V_BATT
- added copper zone on F.Cu, net unconnected-(IC3-SYNCOUT_1-Pad17)
Other:
- board size 54.5 x 139.7 mm -> 198.1 x 139.7 mm
