File: Hardware/OM_Landroid_MB/OM Landroid MB.kicad_sch (KiCad schematic)
At the start: 6 parts

Commit message: Weekend progress
Other:
- sheet IMU ports: added none; removed RX, TX
Changed lines of the file:
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@@
 (kicad_sch (version 20230121) (generator eeschema)
   (paper "A3")
-  (junction (at 186.055 147.32) (diameter 0) (color 0 0 0 0)
-  )
   (junction (at 101.6 151.765) (diameter 0) (color 0 0 0 0)
   )
@@
   )
   (junction (at 98.425 161.925) (diameter 0) (color 0 0 0 0)
-  )
-  (junction (at 188.595 149.86) (diameter 0) (color 0 0 0 0)
   )
   (no_connect (at 367.03 92.075))
@@
     (stroke (width 0) (type default))
   )
-  (wire (pts (xy 188.595 149.86) (xy 191.77 149.86))
-    (stroke (width 0) (type default))
-  )
-  (wire (pts (xy 188.595 149.86) (xy 188.595 142.24))
-    (stroke (width 0) (type default))
-  )
   (wire (pts (xy 243.84 173.99) (xy 243.84 181.61))
     (stroke (width 0) (type default))
@@
     (stroke (width 0) (type default))
   )
-  (wire (pts (xy 170.815 147.32) (xy 186.055 147.32))
-    (stroke (width 0) (type default))
-  )
   (wire (pts (xy 101.6 151.765) (xy 132.715 151.765))
     (stroke (width 0) (type default))
@@
     (stroke (width 0) (type default))
   )
-  (wire (pts (xy 170.815 149.86) (xy 188.595 149.86))
+  (wire (pts (xy 170.815 149.86) (xy 191.77 149.86))
     (stroke (width 0) (type default))
   )
@@
     (stroke (width 0) (type default))
   )
-  (wire (pts (xy 186.055 139.7) (xy 191.77 139.7))
-    (stroke (width 0) (type default))
-  )
   (wire (pts (xy 95.25 146.685) (xy 95.25 149.225))
     (stroke (width 0) (type default))
@@
     (stroke (width 0) (type default))
   )
-  (wire (pts (xy 186.055 147.32) (xy 186.055 139.7))
-    (stroke (width 0) (type default))
-  )
   (wire (pts (xy 170.815 191.77) (xy 223.52 191.77))
     (stroke (width 0) (type default))
@@
     (stroke (width 0) (type default))
   )
-  (wire (pts (xy 188.595 142.24) (xy 191.77 142.24))
-    (stroke (width 0) (type default))
-  )
   (wire (pts (xy 68.58 124.46) (xy 132.715 124.46))
     (stroke (width 0) (type default))
   )
-  (wire (pts (xy 186.055 147.32) (xy 191.77 147.32))
+  (wire (pts (xy 170.815 147.32) (xy 191.77 147.32))
     (stroke (width 0) (type default))
   )
@@
       (effects (font (size 1.27 1.27)) (justify left))
     )
-    (pin "RX" input (at 191.77 142.24 180)
-      (effects (font (size 1.27 1.27)) (justify left))
-    )
-    (pin "TX" output (at 191.77 139.7 180)
-      (effects (font (size 1.27 1.27)) (justify left))
-    )

Commit message: Finished Mainboard
Finished Mainboard redesign for OM Landroid
Other:
- sheet RaspberryPi ports: added Display SCL, Display SDA; removed none
- sheet RobotConnectors ports: added Display SCL, Display SDA; removed none

Commit message: Updates and revisions to charging connections
Parts:
- removed R41: 1k, Resistor_SMD:R_0805_2012Metric_Pad1.20x1.40mm_HandSolder, symbol Device:R
Connections:
- net RobotConnectors/V_CHARGE renamed +3V3
- net pico/V_CHARGE renamed RobotConnectors/Battery Temp
Other:
- sheet RobotConnectors ports: added Battery Temp; removed V_CHARGE
- sheet pico ports: added Battery Temp; removed V_CHARGE
- moved on the sheet: R40
Changed lines of the file:
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@@
   (junction (at 101.6 151.765) (diameter 0) (color 0 0 0 0)
   )
-  (junction (at 95.25 149.225) (diameter 0) (color 0 0 0 0)
-  )
-  (junction (at 98.425 161.925) (diameter 0) (color 0 0 0 0)
+  (junction (at 95.25 147.574) (diameter 0) (color 0 0 0 0)
   )
   (no_connect (at 367.03 92.075))
@@
     (stroke (width 0) (type default))
   )
+  (wire (pts (xy 84.074 141.986) (xy 84.074 144.018))
+    (stroke (width 0) (type default))
+  )
   (wire (pts (xy 175.26 144.78) (xy 175.26 129.54))
     (stroke (width 0) (type default))
@@
     (stroke (width 0) (type default))
   )
-  (wire (pts (xy 95.25 137.795) (xy 95.25 139.065))
-    (stroke (width 0) (type default))
-  )
   (wire (pts (xy 68.58 229.235) (xy 85.725 229.235))
     (stroke (width 0) (type default))
   )
-  (wire (pts (xy 68.58 137.795) (xy 95.25 137.795))
-    (stroke (width 0) (type default))
-  )
   (wire (pts (xy 248.412 181.61) (xy 248.412 172.212))
     (stroke (width 0) (type default))
@@
     (stroke (width 0) (type default))
   )
+  (wire (pts (xy 68.58 147.574) (xy 95.25 147.574))
+    (stroke (width 0) (type default))
+  )
+  (wire (pts (xy 95.25 144.018) (xy 95.25 147.574))
+    (stroke (width 0) (type default))
+  )
   (wire (pts (xy 83.82 231.775) (xy 68.58 231.775))
     (stroke (width 0) (type default))
   )
-  (wire (pts (xy 95.25 149.225) (xy 95.25 153.035))
-    (stroke (width 0) (type default))
-  )
   (wire (pts (xy 268.097 197.866) (xy 272.796 197.866))
     (stroke (width 0) (type default))
@@
     (stroke (width 0) (type default))
   )
-  (wire (pts (xy 95.25 160.655) (xy 95.25 161.925))
-    (stroke (width 0) (type default))
-  )
   (wire (pts (xy 68.58 204.47) (xy 132.715 204.47))
     (stroke (width 0) (type default))
@@
     (stroke (width 0) (type default))
   )
-  (wire (pts (xy 95.25 146.685) (xy 95.25 149.225))
+  (wire (pts (xy 84.074 144.018) (xy 87.376 144.018))
     (stroke (width 0) (type default))
   )
@@
     (stroke (width 0) (type default))
   )
+  (wire (pts (xy 94.996 144.018) (xy 95.25 144.018))
+    (stroke (width 0) (type default))
+  )
   (wire (pts (xy 245.872 181.61) (xy 245.872 173.228))
     (stroke (width 0) (type default))
@@
     (stroke (width 0) (type default))
   )
+  (wire (pts (xy 95.25 147.574) (xy 95.25 149.225))
+    (stroke (width 0) (type default))
+  )
   (wire (pts (xy 123.19 144.145) (xy 123.19 132.08))
     (stroke (width 0) (type default))
@@
   )
   (wire (pts (xy 253.492 120.65) (xy 253.492 181.61))
-    (stroke (width 0) (type default))
-  )
-  (wire (pts (xy 95.25 161.925) (xy 98.425 161.925))
     (stroke (width 0) (type default))
   )
@@
     )
   )
-  (symbol (lib_id "Device:R") (at 95.25 156.845 180) (unit 1)
-    (in_bom yes) (on_board yes) (dnp no) (fields_autoplaced)
-    (property "Reference" "R41" (at 97.028 155.9365 0)
-      (effects (font (size 1.27 1.27)) (justify right))
-    )
-    (property "Value" "1k" (at 97.028 158.7116 0)
-      (effects (font (size 1.27 1.27)) (justify right))
-    )
-    (property "Footprint" "Resistor_SMD:R_0805_2012Metric_Pad1.20x1.40mm_HandSolder" (at 97.028 156.845 90)
-      (effects (font (size 1.27 1.27)) hide)
-    )
-    (property "Datasheet" "~" (at 95.25 156.845 0)
-      (effects (font (size 1.27 1.27)) hide)
-    )
-    (property "Stock_PN" "R-805-1K-.125W-1%" (at 95.25 156.845 0)
-      (effects (font (size 1.27 1.27)) hide)
-    )
-    (property "Digikey" "311-1.00KCRCT-ND" (at 95.25 156.845 0)
-      (effects (font (size 1.27 1.27)) hide)
-    )
-    (property "Part Number" "RC0805FR-071KL" (at 95.25 156.845 0)
-      (effects (font (size 1.27 1.27)) hide)
-    )
-    (property "LCSC" "C95781" (at 95.25 156.845 0)
-      (effects (font (size 1.27 1.27)) hide)
-    )
-    (pin "1")
-    (pin "2")
-    (instances
-      (project "OM Landroid MB"
-        (path "/c454102f-dc92-4550-9492-797fc8e6b49c"
-          (reference "R41") (unit 1)
-        )
-      )
-    )
-  )
   (symbol (lib_id "power:+5V") (at 325.755 193.04 0) (unit 1)
     (in_bom yes) (on_board yes) (dnp no) (fields_autoplaced)
@@
     )
   )
-  (symbol (lib_id "Device:R") (at 95.25 142.875 180) (unit 1)
+  (symbol (lib_id "Device:R") (at 91.186 144.018 270) (unit 1)
     (in_bom yes) (on_board yes) (dnp no) (fields_autoplaced)
-    (property "Reference" "R40" (at 97.028 141.9665 0)
-      (effects (font (size 1.27 1.27)) (justify right))
-    )
-    (property "Value" "10k" (at 97.028 144.7416 0)
-      (effects (font (size 1.27 1.27)) (justify right))
-    )
-    (property "Footprint" "Resistor_SMD:R_0805_2012Metric_Pad1.20x1.40mm_HandSolder" (at 97.028 142.875 90)
-      (effects (font (size 1.27 1.27)) hide)
-    )
-    (property "Datasheet" "~" (at 95.25 142.875 0)
-      (effects (font (size 1.27 1.27)) hide)
-    )
-    (property "Digikey" "738-RMCF0805FG10K0CT-ND" (at 95.25 142.875 0)
-      (effects (font (size 1.27 1.27)) hide)
-    )
-    (property "Part Number" "RMCF0805FG10K0" (at 95.25 142.875 0)
-      (effects (font (size 1.27 1.27)) hide)
-    )
-    (property "Stock_PN" "R-805-10K-.125W-1%" (at 95.25 142.875 0)
-      (effects (font (size 1.27 1.27)) hide)
-    )
-    (property "LCSC" "C17414" (at 95.25 142.875 0)
+    (property "Reference" "R40" (at 91.186 138.303 90)
+      (effects (font (size 1.27 1.27)))
+    )
+    (property "Value" "10k" (at 91.186 140.843 90)
+      (effects (font (size 1.27 1.27)))
+    )
+    (property "Footprint" "Resistor_SMD:R_0805_2012Metric_Pad1.20x1.40mm_HandSolder" (at 91.186 142.24 90)
+      (effects (font (size 1.27 1.27)) hide)
+    )
+    (property "Datasheet" "~" (at 91.186 144.018 0)
+      (effects (font (size 1.27 1.27)) hide)
+    )
+    (property "Digikey" "738-RMCF0805FG10K0CT-ND" (at 91.186 144.018 0)
+      (effects (font (size 1.27 1.27)) hide)
+    )
+    (property "Part Number" "RMCF0805FG10K0" (at 91.186 144.018 0)
+      (effects (font (size 1.27 1.27)) hide)
+    )
+    (property "Stock_PN" "R-805-10K-.125W-1%" (at 91.186 144.018 0)
+      (effects (font (size 1.27 1.27)) hide)
+    )
+    (property "LCSC" "C17414" (at 91.186 144.018 0)
       (effects (font (size 1.27 1.27)) hide)
     )
@@
         (path "/c454102f-dc92-4550-9492-797fc8e6b49c"
           (reference "R18") (unit 1)
+        )
+      )
+    )
+  )
+  (symbol (lib_id "power:+3V3") (at 84.074 141.986 0) (unit 1)
+    (in_bom yes) (on_board yes) (dnp no) (fields_autoplaced)
+    (property "Reference" "#PWR03" (at 84.074 145.796 0)
+      (effects (font (size 1.27 1.27)) hide)
+    )
+    (property "Value" "+3V3" (at 84.074 137.16 0)
+      (effects (font (size 1.27 1.27)))
+    )
+    (property "Footprint" "" (at 84.074 141.986 0)
+      (effects (font (size 1.27 1.27)) hide)
+    )
+    (property "Datasheet" "" (at 84.074 141.986 0)
+      (effects (font (size 1.27 1.27)) hide)
+    )
+    (pin "1")
+    (instances
+      (project "OM Landroid MB"
+        (path "/c454102f-dc92-4550-9492-797fc8e6b49c"
+          (reference "#PWR03") (unit 1)
         )
       )
@@
       (effects (font (size 1.27 1.27)) (justify right))
     )
-    (pin "V_CHARGE" output (at 68.58 137.795 0)
-      (effects (font (size 1.27 1.27)) (justify right))
-    )
     (pin "ML_P3" input (at 68.58 83.82 0)
       (effects (font (size 1.27 1.27)) (justify right))
@@
     )
     (pin "Display SDA" bidirectional (at 68.58 240.538 0)
+      (effects (font (size 1.27 1.27)) (justify right))
+    )
+    (pin "Battery Temp" output (at 68.58 147.574 0)
       (effects (font (size 1.27 1.27)) (justify right))
     )
@@
       (effects (font (size 1.27 1.27)) (justify left))
     )
-    (pin "V_CHARGE" input (at 132.715 149.225 180)
-      (effects (font (size 1.27 1.27)) (justify left))
-    )
     (pin "V_IN" input (at 132.715 151.765 180)
       (effects (font (size 1.27 1.27)) (justify left))
@@
       (effects (font (size 1.27 1.27)) (justify right))
     )
-    (instances
+    (pin "Battery Temp" input (at 132.715 149.225 180)
+      (effects (font (size 1.27 1.27)) (justify left))
+    )
+    (instances
