File: Hardware/OM_Landroid_MB/pico.kicad_sch (KiCad schematic)
At the start: 7 parts, among them U10 74HC4051, U11 Pico, U7 SN74LV1T34DBV, U9 74HC4051

Commit message: Update 21.11.23
Parts:
- U11: footprint PicoW:Raspberry_Pi_Pico_SMT_THT -> PicoW:Raspberry_Pi_Pico_THT
Changed lines of the file:
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@@
       (effects (font (size 1.27 1.27)))
     )
-    (property "Footprint" "PicoW:Raspberry_Pi_Pico_SMT_THT" (at 215.9 87.63 0)
+    (property "Footprint" "PicoW:Raspberry_Pi_Pico_THT" (at 215.9 87.63 0)
       (effects (font (size 1.27 1.27)) hide)
     )

Commit message: Updates and revisions to charging connections
Connections:
- net V_CHARGE renamed Battery Temp
Changed lines of the file:
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@@
     (effects (font (size 1.27 1.27)) (justify left bottom))
-  )
-  (hierarchical_label "V_CHARGE" (shape input) (at 254 87.63 0) (fields_autoplaced)
-    (effects (font (size 1.27 1.27)) (justify left))
   )
   (hierarchical_label "IMU_SCK" (shape output) (at 173.99 87.63 180) (fields_autoplaced)
@@
     (effects (font (size 1.27 1.27)) (justify right))
   )
+  (hierarchical_label "Battery Temp" (shape input) (at 254 87.63 0) (fields_autoplaced)
+    (effects (font (size 1.27 1.27)) (justify left))
+  )
   (hierarchical_label "SWCLK" (shape input) (at 215.9 130.81 270) (fields_autoplaced)
