File: Hardware/OM_Landroid_MB/RaspberryPi.kicad_sch (KiCad schematic)
At the start: 13 parts, among them J21 Raspberry_Pi_2_3, J22 Conn_02x04_Odd_Even, M1 Fan, Q3 BSS138, SW1 MK-11C04-G013, U3 SIP32509DT

Commit message: Weekend progress
Parts:
- J21: footprint RPi_c:RPi_40Pin_Fan_Courtyard -> Connector_PinSocket_2.54mm:PinSocket_2x20_P2.54mm_Vertical
Changed lines of the file:
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@@
       (effects (font (size 1.27 1.27)) (justify left))
     )
-    (property "Footprint" "RPi_c:RPi_40Pin_Fan_Courtyard" (at 107.315 133.985 0)
+    (property "Footprint" "Connector_PinSocket_2.54mm:PinSocket_2x20_P2.54mm_Vertical" (at 107.315 133.985 0)
       (effects (font (size 1.27 1.27)) hide)
     )

Commit message: Finished Mainboard
Finished Mainboard redesign for OM Landroid
Connections:
- net Display SDA: now reaches J21.3 (SDA/GPIO2)
- net Display SCL: now reaches J21.5 (SCL/GPIO3)
- no-connect marks 18 -> 16
Changed lines of the file:
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@@
   (no_connect (at 149.86 35.56))
   (no_connect (at 149.86 33.02))
-  (no_connect (at 127.635 121.285))
-  (no_connect (at 127.635 118.745))
   (no_connect (at 112.395 100.965))
   (no_connect (at 109.855 100.965))
@@
     (effects (font (size 1.27 1.27)) (justify left))
   )
+  (hierarchical_label "Display SCL" (shape output) (at 127.635 121.285 0) (fields_autoplaced)
+    (effects (font (size 1.27 1.27)) (justify left))
+  )
   (hierarchical_label "UART1_TXD" (shape output) (at 158.115 111.125 0) (fields_autoplaced)
     (effects (font (size 1.27 1.27)) (justify left))
@@
     (effects (font (size 1.27 1.27)) (justify right))
   )
+  (hierarchical_label "Display SDA" (shape bidirectional) (at 127.635 118.745 0) (fields_autoplaced)
+    (effects (font (size 1.27 1.27)) (justify left))
+  )
   (symbol (lib_id "power:+5V") (at 199.39 20.32 0) (unit 1)

Commit message: Changes to align BOM with board
Changes were needed to  align the BOM content with the board and to reflect component availability from Digikey
Parts:
- J21: value Raspberry_Pi_2_3 -> Extended GPIO Header Female; Digikey S5729-ND -> 1568-PRT-16764-ND
Changed lines of the file:
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@@
       (effects (font (size 1.27 1.27)) (justify left))
     )
-    (property "Value" "Raspberry_Pi_2_3" (at 114.4144 100.965 0)
+    (property "Value" "Extended GPIO Header Female" (at 114.4144 100.965 0)
       (effects (font (size 1.27 1.27)) (justify left))
     )
@@
       (effects (font (size 1.27 1.27)) hide)
     )
-    (property "Digikey" "S5729-ND" (at 107.315 133.985 0)
+    (property "Digikey" "1568-PRT-16764-ND" (at 107.315 133.985 0)
       (effects (font (size 1.27 1.27)) hide)
     )
